File: esp8266.sch (KiCad schematic (older format))
At the start: 1 part

Commit message: first commit
kicad
Parts:
- removed U?: ESP-07v2, symbol ESP-07v2
- added C1, C2, C3, C5, C6: C, symbol C
- added C4, C7: CP, symbol CP
- added D1, D2, D3: LED_Small, symbol LED_Small
- added J1, J3: CONN_01X02, symbol CONN_01X02
- added J2, J_DHT1, J_PIR1, J_Serial1: CONN_01X03, symbol CONN_01X03
- added J_Sw1: HEADER_3, symbol HEADER_3
- added K1, K2: Omron_G3MB-202P, symbol Omron_G3MB-202P
- added Q1, Q2: BC548, TO_SOT_Packages_THT:TO-92_Molded_Narrow, symbol BC548
- added R1, R10, R11, R12, R13, R2, R3, R4, R5, R6, R7, R8, R9: R, symbol R
- added SW_P1, SW_R1: SW_PUSH, symbol SW_PUSH
- added U1: ESP-07v2, symbol ESP-07v2
- added U11: HiLink_HLK_PM01, symbol HiLink_HLK_PM01
- added U2: LM1117-3.3, symbol LM1117-3.3
Connections:
- new net: D3.2 (A), R13.2
- new net: D3.1 (K), K2.4 (input-), Q2.1 (C)
- new net: D2.1 (K), K1.4 (input-), Q1.1 (C)
- new net: D2.2 (A), R12.2
- new net: Q1.2 (B), R10.1
- new net: Q2.2 (B), R11.1
- new net: R9.1, U1.10 (GPIO15)
- new net: R4.1, R6.2, U1.2 (ADC)
- new net: R7.1, U1.3 (CH_PD)
- new net +3.3V: C3.2, C6.1, C7.1, J_DHT1.3 (P3), R1.1, R2.1, R3.1, R5.1, R7.2, R8.1, U1.8 (VCC), U2.2 (VO), U2.4 (VO)
- new net +5V: C4.1, C5.1, J_PIR1.3 (P3), K1.3 (input+), K2.3 (input+), R12.1, R13.1, U2.3 (VI)
- new net An: J3.2 (P2), R4.2
- new net DHT: J_DHT1.2 (P2), U1.11 (GPIO2)
- new net GND: C1.2, C2.2, C3.1, C4.2, C5.2, C6.2, C7.2, D1.1 (K), J3.1 (P1), J_DHT1.1 (P1), J_PIR1.1 (P1), J_Serial1.1 (P1), J_Sw1.1, Q1.3 (E), Q2.3 (E), R6.1, R9.2, SW_P1.1, SW_R1.1, U1.9 (GND), U2.1 (GND/ADJ)
- new net L_1: J2.2 (P2), K1.2 (load)
- new net L_2: J2.3 (P3), K2.2 (load)
- new net Led: D1.2 (A), R3.2, U1.4 (GPIO16)
- new net Lin: J1.2 (P2), J2.1 (P1), K1.1 (load), K2.1 (load)
- new net Neu: J1.1 (P1)
- new net PIR: J_PIR1.2 (P2), U1.5 (GPIO14)
- new net Prog: R2.2, SW_P1.2, U1.12 (GPIO0)
- new net Rel_K1: R10.2, U1.14 (GPIO5)
- new net Rel_K2: R11.2, U1.13 (GPIO4)
- new net Reset: R1.2, SW_R1.2, U1.1 (REST)
- new net Rx: J_Serial1.2 (P2), U1.15 (RXD)
- new net Sw_1: C1.1, J_Sw1.2, R5.2, U1.6 (GPIO12)
- new net Sw_2: C2.1, J_Sw1.3, R8.2, U1.7 (GPIO13)
- new net Tx: J_Serial1.3 (P3), U1.16 (TXD)

Commit message: add
Parts:
- removed U2: LM1117-3.3, symbol LM1117-3.3
- added U2: LM1117-SOT, TO_SOT_Packages_SMD:SOT-223-3Lead_TabPin2, symbol LM1117-SOT
- C1, C2, C3, C5, C6: footprint (none) -> Capacitors_THT:C_Disc_D3.4mm_W2.1mm_P2.50mm
- C4, C7: footprint (none) -> w_capacitors:CP_5x7mm
- D1, D2, D3: footprint (none) -> LEDs:LED_D5.0mm
- J1, J3: footprint (none) -> Pin_Headers:Pin_Header_Straight_1x02_Pitch2.54mm
- J2, J_DHT1, J_PIR1, J_Serial1: footprint (none) -> Pin_Headers:Pin_Header_Straight_1x03_Pitch2.54mm
- J_Sw1, SW_P1, SW_R1: footprint (none) -> Buttons_Switches_SMD:SW_DIP_x1_W5.08mm_Slide_Copal_CHS-A
- R1, R10, R11, R12, R13, R2, R3, R4, R5, R6, R7, R8, R9: footprint (none) -> Resistors_THT:R_Axial_DIN0204_L3.6mm_D1.6mm_P7.62mm_Horizontal
- U1: footprint (none) -> ESP8266:ESP-07v2
Connections:
- net +3.3V: now also C3.1, U2.2 (VOUT); no longer C3.2
- net +5V: now also U11.3 (V+), U2.3 (VIN)
- net GND: now also C3.2, U11.4 (V-), U2.1 (ADJ/GND); no longer C3.1
- net Lin: now also U11.1 (AC-P)
- net Neu: now also U11.2 (AC-N)
Other:
- moved on the sheet: C3, C4, C5, C6, C7, R4, R6, R7, R9, U1
